Commit message: ..

File: roscue_arm_description/urdf/assemblies/roscue_arm.urdf.xacro (robot description, xacro)
@@ -3,5 +3,5 @@
   <xacro:macro name="roscue_arm" params="prefix">
     <!-- Links -->
-    <link name="${prefix}base_link">
+    <link name="${prefix}arm_base_link">
       <inertial>
         <origin xyz="0.085592 -0.000006 0.033051" rpy="0 0 0"/>
@@ -131,5 +131,5 @@
     <!-- Joints (internal to assembly) -->
     <joint name="${prefix}base_joint" type="revolute">
-      <parent link="${prefix}base_link"/>
+      <parent link="${prefix}arm_base_link"/>
       <child link="${prefix}first_link"/>
       <origin xyz="0.000000 0.000000 0.027000" rpy="0.000000 -0.000000 0.000000"/>
@@ -142,5 +142,5 @@
       <origin xyz="-0.065000 0.000000 0.063000" rpy="0.000000 -1.570796 0.000000"/>
       <axis xyz="-0.000000 -0.000000 -1.000000"/>
-      <limit lower="-1.4835" upper="1.5708" effort="100.0" velocity="1.00"/>
+      <limit lower="-1.5097" upper="1.5708" effort="100.0" velocity="1.00"/>
     </joint>
     <joint name="${prefix}arm_joint_2" type="revolute">

File: roscue_arm_description/urdf/roscue_arm.urdf (robot description, URDF)
Before this commit: robot roscue_arm, 15 links, 14 joints
Links:
- added link arm_base_link, mass 2.059958; collision mesh filename=package://roscue_arm_description/meshes/roscue_arm/base_lin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 scale=1 1 1; visual mesh filename=package://roscue_arm_description/meshes/roscue_arm/base_lin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 scale=1 1 1
- added link button_contact_link
- added link camera_link; collision box size=0.090 0.025 0.025; visual box size=0.090 0.025 0.025
- added link grasp_tcp_link
- link base_link: mass 2.059958 -> None; geometry 
Joints:
- added joint arm_mount_joint: type fixed, parent base_link, child arm_base_link, origin xyz=-0.295 0.075 0.665 rpy=0 0 0
- added joint button_contact_joint: type fixed, parent gripper_base_link, child button_contact_link, origin xyz=-0.073434 -0.044148 0.179650 rpy=0 0 0.52359878
- added joint camera_mount_joint: type fixed, parent gripper_base_link, child camera_link, origin xyz=0.0 -0.070 0.057 rpy=1.57079633 -1.57079633 0.0
- added joint grasp_tcp_joint: type fixed, parent gripper_base_link, child grasp_tcp_link, origin xyz=0 0 0.134295 rpy=0 0 0
- joint arm_joint_1: limit effort=100.0 velocity=1.00 -> lower=-1.5097 upper=1.5708 effort=100.0 velocity=1.00; type continuous -> revolute
- joint arm_joint_2: limit effort=100.0 velocity=1.00 -> lower=-1.3631 upper=1.3963 effort=100.0 velocity=1.00; type continuous -> revolute
- joint arm_joint_3: limit effort=100.0 velocity=1.00 -> lower=-1.5970 upper=1.5708 effort=100.0 velocity=1.00; type continuous -> revolute
- joint arm_joint_4: limit effort=100.0 velocity=1.00 -> lower=-1.5708 upper=1.5708 effort=100.0 velocity=1.00; type continuous -> revolute
- joint base_joint: limit effort=100.0 velocity=1.00 -> lower=-1.5708 upper=3.1416 effort=100.0 velocity=1.00; parent base_link -> arm_base_link; type continuous -> revolute
- joint finger_1_base_joint: limit effort=100.0 velocity=1.00 -> lower=-1.2269 upper=1.2269 effort=100.0 velocity=1.00; type continuous -> revolute
- joint finger_1_middle_joint: limit effort=100.0 velocity=1.00 -> lower=-2.4033 upper=0.9198 effort=100.0 velocity=1.00; type continuous -> revolute
- joint finger_1_tip_joint: limit effort=100.0 velocity=1.00 -> lower=-1.9426 upper=1.9426 effort=100.0 velocity=1.00; type continuous -> revolute
- joint finger_2_base_joint: limit effort=100.0 velocity=1.00 -> lower=-1.2269 upper=1.2269 effort=100.0 velocity=1.00; type continuous -> revolute
- joint finger_2_middle_joint: limit effort=100.0 velocity=1.00 -> lower=-2.4033 upper=0.9198 effort=100.0 velocity=1.00; type continuous -> revolute
- joint finger_2_tip_joint: limit effort=100.0 velocity=1.00 -> lower=-1.9426 upper=1.9426 effort=100.0 velocity=1.00; type continuous -> revolute
- joint finger_3_base_joint: limit effort=100.0 velocity=1.00 -> lower=-1.2269 upper=1.2269 effort=100.0 velocity=1.00; type continuous -> revolute
- joint finger_3_middle_joint: limit effort=100.0 velocity=1.00 -> lower=-2.4033 upper=0.9198 effort=100.0 velocity=1.00; type continuous -> revolute
- joint finger_3_tip_joint: limit effort=100.0 velocity=1.00 -> lower=-1.9426 upper=1.9426 effort=100.0 velocity=1.00; type continuous -> revolute

File: roscue_arm_description/urdf/roscue_arm.urdf.xacro (robot description, xacro)
@@ -33,4 +33,15 @@
   <xacro:finger_2_base_link prefix=""/>
   <xacro:roscue_arm prefix=""/>
+  <!--
+    Mobile-platform mount measured in the final integration PDF.
+    The mobile robot owns base_link and publishes odom -> base_link; this
+    robot_state_publisher only adds the arm subtree below it.
+  -->
+  <link name="base_link"/>
+  <joint name="arm_mount_joint" type="fixed">
+    <parent link="base_link"/>
+    <child link="arm_base_link"/>
+    <origin xyz="-0.295 0.075 0.665" rpy="0 0 0"/>
+  </joint>
   <!-- Mount joints (cross-assembly connections) -->
   <joint name="finger_1_base_joint" type="revolute">
@@ -187,7 +198,7 @@
   </ros2_control>
   <!--
-    RealSense wrist mount. The camera driver owns camera_link's optical-frame
-    children; robot_state_publisher only connects the camera to the arm.
-    Replace this provisional transform after measuring the physical mount.
+    RealSense wrist mount measured in the final integration PDF. The camera
+    driver owns camera_link's optical-frame children; robot_state_publisher
+    only connects the camera root to the arm.
   -->
   <link name="camera_link">
@@ -211,5 +222,22 @@
     <parent link="gripper_base_link"/>
     <child link="camera_link"/>
-    <origin xyz="0.0 0.0 0.07" rpy="0.0 0.0 0.0"/>
+    <origin xyz="0.0 -0.070 0.057" rpy="1.57079633 -1.57079633 0.0"/>
+  </joint>
+  <!-- Fixed button TCP: third-finger contact point from the final PDF. -->
+  <link name="button_contact_link"/>
+  <joint name="button_contact_joint" type="fixed">
+    <parent link="gripper_base_link"/>
+    <child link="button_contact_link"/>
+    <origin xyz="-0.073434 -0.044148 0.179650" rpy="0 0 0.52359878"/>
+  </joint>
+  <!--
+    Center of the three fingertip-joint origins at the configured closed
+    object pose. Pick targets use this TCP instead of the palm origin.
+  -->
+  <link name="grasp_tcp_link"/>
+  <joint name="grasp_tcp_joint" type="fixed">
+    <parent link="gripper_base_link"/>
+    <child link="grasp_tcp_link"/>
+    <origin xyz="0 0 0.134295" rpy="0 0 0"/>
   </joint>
 </robot>
